File: Convolution Thing/Display.sch (KiCad schematic (older format))
At the start: 0 parts

Commit message: Better CV inputs, LED driver, display & USB interfaces
Parts:
- added C? (x2): 2.2uF, symbol Device:C
- added C?: 100nF, symbol Device:C
- added DS?: EA_OLEDM128-6GGA, EAOLEDM1286GGA, symbol SamacSys:EA_OLEDM128-6GGA
- added R?: 910k, symbol Device:R
Connections:
- new net +12V: C?.1, DS?.21 (VCC_1), DS?.22 (VCC_2), DS?.39 (VCC_3), DS?.40 (VCC_4)
- new net +3V3: C?.1, DS?.25 (VDD), DS?.26 (BS0)
- new net DISPLAY_SCL: DS?.32 (D0)
- new net DISPLAY_SDA: DS?.33 (D1), DS?.34 (D2)
- new net GND: C?.2, C?.2, C?.2, DS?.1 (ESD_GND_1), DS?.20 (ESD_GND_2), DS?.23 (GND_1), DS?.24 (GND_2), DS?.27 (BS1), DS?.28 (GND_3), DS?.29 (CS), DS?.30 (RES), DS?.31 (D/C), DS?.35 (GND_4), R?.2
- new net IREF: DS?.36 (IREF), R?.1
- new net VCOMH: C?.1, DS?.37 (VCOMH_1), DS?.38 (VCOMH_2)
- no-connect marks 0 -> 4
Other:
- note added: "I2C Address"
- note added: "I2C Interface"
- note added: "I2C Mode"
