File: Convolution Thing/Audio In.sch (KiCad schematic (older format))
At the start: 16 parts, among them J6 In Left, J7 In Right, U5 NE5532, U6 NE5532

Commit message: PCB layout work and related changes to the schematic
Parts:
- J5: renamed from J6; footprint SamacSys:ACJMNV352S -> Connector_Audio:Jack_3.5mm_QingPu_WQP-PJ398SM_Vertical_CircularHoles
- J6: renamed from J7; footprint SamacSys:ACJMNV352S -> Connector_Audio:Jack_3.5mm_QingPu_WQP-PJ398SM_Vertical_CircularHoles
- TP10: renamed from TP16; value IN L TP -> IN R TP
- renumbered C27 to C23, C28 to C24, C29 to C25, C30 to C26, C31 to C27, C32 to C28, R18 to R16, R19 to R17, R20 to R18, R21 to R19, TP15 to TP9, U5 to U4, U6 to U4
Connections:
- net ADC_VIN_L renamed CODEC_VIN_L
- net ADC_VIN_R renamed CODEC_VIN_R
Changed lines of the file:
@@
 $Descr A4 11693 8268
 encoding utf-8
-Sheet 7 13
+Sheet 6 13
 Title ""
 Date ""
@@
 $EndDescr
 $Comp
-L Connector:AudioJack2_SwitchT J6
+L Connector:AudioJack2_SwitchT J5
 U 1 1 61066301
 P 900 1450
-F 0 "J6" H 721 1383 50  0000 R CNN
+F 0 "J5" H 721 1383 50  0000 R CNN
 F 1 "In Left" H 1050 1150 50  0000 R CNN
-F 2 "SamacSys:ACJMNV352S" H 900 1450 50  0001 C CNN
+F 2 "Connector_Audio:Jack_3.5mm_QingPu_WQP-PJ398SM_Vertical_CircularHoles" H 900 1450 50  0001 C CNN
 F 3 "~" H 900 1450 50  0001 C CNN
 	1    900  1450
@@
 $EndComp
 $Comp
-L power:GND #PWR052
+L power:GND #PWR039
 U 1 1 6106718A
 P 1100 1550
-F 0 "#PWR052" H 1100 1300 50  0001 C CNN
+F 0 "#PWR039" H 1100 1300 50  0001 C CNN
 F 1 "GND" H 1105 1377 50  0000 C CNN
 F 2 "" H 1100 1550 50  0001 C CNN
@@
 $EndComp
 $Comp
-L Amplifier_Operational:NE5532 U5
+L Amplifier_Operational:NE5532 U4
 U 3 1 6108EB84
 P 7100 1300
-F 0 "U5" H 7058 1346 50  0000 L CNN
+F 0 "U4" H 7058 1346 50  0000 L CNN
 F 1 "NE5532" H 7058 1255 50  0000 L CNN
 F 2 "Package_SO:SOIC-8_3.9x4.9mm_P1.27mm" H 7100 1300 50  0001 C CNN
@@
 $EndComp
 $Comp
-L power:+12V #PWR056
+L power:+12V #PWR043
 U 1 1 610913E7
 P 7000 1000
-F 0 "#PWR056" H 7000 850 50  0001 C CNN
+F 0 "#PWR043" H 7000 850 50  0001 C CNN
 F 1 "+12V" H 7150 1050 50  0000 C CNN
 F 2 "" H 7000 1000 50  0001 C CNN
@@
 $EndComp
 $Comp
-L power:-12V #PWR057
+L power:-12V #PWR044
 U 1 1 6109183E
 P 7000 1600
-F 0 "#PWR057" H 7000 1700 50  0001 C CNN
+F 0 "#PWR044" H 7000 1700 50  0001 C CNN
 F 1 "-12V" H 6850 1650 50  0000 C CNN
 F 2 "" H 7000 1600 50  0001 C CNN
@@
 Connection ~ 7000 1000
 $Comp
-L Device:C C32
+L Device:C C28
 U 1 1 61096E23
 P 6750 1600
-F 0 "C32" V 6498 1600 50  0000 C CNN
+F 0 "C28" V 6498 1600 50  0000 C CNN
 F 1 "100nF" V 6589 1600 50  0000 C CNN
 F 2 "Capacitor_SMD:C_0805_2012Metric" H 6788 1450 50  0001 C CNN
@@
 $EndComp
 $Comp
-L power:GND #PWR055
+L power:GND #PWR042
 U 1 1 61096E29
 P 6500 1600
-F 0 "#PWR055" H 6500 1350 50  0001 C CNN
+F 0 "#PWR042" H 6500 1350 50  0001 C CNN
 F 1 "GND" H 6505 1427 50  0000 C CNN
 F 2 "" H 6500 1600 50  0001 C CNN
@@
 Connection ~ 7000 1600
 $Comp
-L Device:C C31
+L Device:C C27
 U 1 1 61093C0F
 P 6750 1000
-F 0 "C31" V 6498 1000 50  0000 C CNN
+F 0 "C27" V 6498 1000 50  0000 C CNN
 F 1 "100nF" V 6589 1000 50  0000 C CNN
 F 2 "Capacitor_SMD:C_0805_2012Metric" H 6788 850 50  0001 C CNN
@@
 $EndComp
 $Comp
-L power:GND #PWR054
+L power:GND #PWR041
 U 1 1 61095461
 P 6500 1000
-F 0 "#PWR054" H 6500 750 50  0001 C CNN
+F 0 "#PWR041" H 6500 750 50  0001 C CNN
 F 1 "GND" H 6505 827 50  0000 C CNN
 F 2 "" H 6500 1000 50  0001 C CNN
@@
 	6500 1000 6600 1000
 $Comp
-L Device:R R18
+L Device:R R16
 U 1 1 610C039D
 P 1800 1450
-F 0 "R18" V 1700 1450 50  0000 C CNN
+F 0 "R16" V 1700 1450 50  0000 C CNN
 F 1 "100k" V 1800 1450 50  0000 C CNN
 F 2 "Resistor_SMD:R_0805_2012Metric" V 1730 1450 50  0001 C CNN
@@
 Connection ~ 1200 1450
 Text GLabel 2750 1550 2    50   Output ~ 0
-ADC_VIN_L
+CODEC_VIN_L
 NoConn ~ 1100 1350
 Wire Wire Line
 	2700 1550 2750 1550
 $Comp
-L Device:C C27
+L Device:C C23
 U 1 1 610D621F
 P 1500 1450
-F 0 "C27" V 1248 1450 50  0000 C CNN
+F 0 "C23" V 1248 1450 50  0000 C CNN
 F 1 "10uF" V 1339 1450 50  0000 C CNN
 F 2 "Capacitor_SMD:C_0805_2012Metric" H 1538 1300 50  0001 C CNN
@@
 $EndComp
 $Comp
-L Connector:TestPoint TP15
+L Connector:TestPoint TP9
 U 1 1 610FCF8B
 P 2700 1550
-F 0 "TP15" H 2450 1700 50  0000 L CNN
+F 0 "TP9" H 2450 1700 50  0000 L CNN
 F 1 "IN L TP" H 2550 1800 50  0000 L CNN
 F 2 "TestPoint:TestPoint_Loop_D2.60mm_Drill1.6mm_Beaded" H 2900 1550 50  0001 C CNN
@@
 $EndComp
 $Comp
-L Amplifier_Operational:NE5532 U5
+L Amplifier_Operational:NE5532 U4
 U 1 1 610C49A2
 P 2350 1550
-F 0 "U5" H 2350 1900 50  0000 C CNN
+F 0 "U4" H 2350 1900 50  0000 C CNN
 F 1 "NE5532" H 2350 1800 50  0000 C CNN
 F 2 "Package_SO:SOIC-8_3.9x4.9mm_P1.27mm" H 2350 1550 50  0001 C CNN
@@
 	2000 1650 2050 1650
 $Comp
-L Device:R R19
+L Device:R R17
 U 1 1 610E377B
 P 2350 1250
-F 0 "R19" V 2450 1250 50  0000 C CNN
+F 0 "R17" V 2450 1250 50  0000 C CNN
 F 1 "22k" V 2350 1250 50  0000 C CNN
 F 2 "Resistor_SMD:R_0805_2012Metric" V 2280 1250 50  0001 C CNN
@@
 $EndComp
 $Comp
-L Device:C C28
+L Device:C C24
 U 1 1 610E3C97
 P 2350 1000
-F 0 "C28" V 2098 1000 50  0000 C CNN
+F 0 "C24" V 2098 1000 50  0000 C CNN
 F 1 "330pF" V 2189 1000 50  0000 C CNN
 F 2 "Capacitor_SMD:C_0805_2012Metric" H 2388 850 50  0001 C CNN
@@
 Connection ~ 2700 1550
 $Comp
-L Connector:AudioJack2_SwitchT J7
+L Connector:AudioJack2_SwitchT J6
 U 1 1 610F5CC0
 P 3650 1450
-F 0 "J7" H 3471 1383 50  0000 R CNN
+F 0 "J6" H 3471 1383 50  0000 R CNN
 F 1 "In Right" H 3800 1150 50  0000 R CNN
-F 2 "SamacSys:ACJMNV352S" H 3650 1450 50  0001 C CNN
+F 2 "Connector_Audio:Jack_3.5mm_QingPu_WQP-PJ398SM_Vertical_CircularHoles" H 3650 1450 50  0001 C CNN
 F 3 "~" H 3650 1450 50  0001 C CNN
 	1    3650 1450
@@
 $EndComp
 $Comp
-L power:GND #PWR053
+L power:GND #PWR040
 U 1 1 610F5CC6
 P 3850 1550
-F 0 "#PWR053" H 3850 1300 50  0001 C CNN
+F 0 "#PWR040" H 3850 1300 50  0001 C CNN
 F 1 "GND" H 3855 1377 50  0000 C CNN
 F 2 "" H 3850 1550 50  0001 C CNN
@@
 $EndComp
 $Comp
-L Device:R R20
+L Device:R R18
 U 1 1 610F5CCC
 P 4550 1450
-F 0 "R20" V 4450 1450 50  0000 C CNN
+F 0 "R18" V 4450 1450 50  0000 C CNN
 F 1 "100k" V 4550 1450 50  0000 C CNN
 F 2 "Resistor_SMD:R_0805_2012Metric" V 4480 1450 50  0001 C CNN
@@
 CODEC_VCOM
 Text GLabel 5500 1550 2    50   Output ~ 0
-ADC_VIN_R
+CODEC_VIN_R
 Wire Wire Line
 	5450 1550 5500 1550
 $Comp
-L Device:C C29
+L Device:C C25
 U 1 1 610F5CDB
 P 4250 1450
-F 0 "C29" V 3998 1450 50  0000 C CNN
+F 0 "C25" V 3998 1450 50  0000 C CNN
 F 1 "10uF" V 4089 1450 50  0000 C CNN
 F 2 "Capacitor_SMD:C_0805_2012Metric" H 4288 1300 50  0001 C CNN
@@
 $EndComp
 $Comp
-L Connector:TestPoint TP16
+L Connector:TestPoint TP10
 U 1 1 610F5CE1
 P 5450 1550
-F 0 "TP16" H 5200 1700 50  0000 L CNN
-F 1 "IN L TP" H 5300 1800 50  0000 L CNN
+F 0 "TP10" H 5200 1700 50  0000 L CNN
+F 1 "IN R TP" H 5300 1800 50  0000 L CNN
 F 2 "TestPoint:TestPoint_Loop_D2.60mm_Drill1.6mm_Beaded" H 5650 1550 50  0001 C CNN
 F 3 "~" H 5650 1550 50  0001 C CNN
@@
 $EndComp
 $Comp
-L Amplifier_Operational:NE5532 U6
+L Amplifier_Operational:NE5532 U4
 U 2 1 610F5CE7
 P 5100 1550
-F 0 "U6" H 5100 1900 50  0000 C CNN
+F 0 "U4" H 5100 1900 50  0000 C CNN
 F 1 "NE5532" H 5100 1800 50  0000 C CNN
 F 2 "Package_SO:SOIC-8_3.9x4.9mm_P1.27mm" H 5100 1550 50  0001 C CNN
@@
 	4750 1650 4800 1650
 $Comp
-L Device:R R21
+L Device:R R19
 U 1 1 610F5CEF
 P 5100 1250
-F 0 "R21" V 5200 1250 50  0000 C CNN
+F 0 "R19" V 5200 1250 50  0000 C CNN
 F 1 "22k" V 5100 1250 50  0000 C CNN
 F 2 "Resistor_SMD:R_0805_2012Metric" V 5030 1250 50  0001 C CNN
@@
 $EndComp
 $Comp
-L Device:C C30
+L Device:C C26
 U 1 1 610F5CF5
 P 5100 1000
-F 0 "C30" V 4848 1000 50  0000 C CNN
+F 0 "C26" V 4848 1000 50  0000 C CNN
 F 1 "330pF" V 4939 1000 50  0000 C CNN
 F 2 "Capacitor_SMD:C_0805_2012Metric" H 5138 850 50  0001 C CNN
