File: Convolution Thing/CODEC.sch (KiCad schematic (older format))
At the start: 7 parts, among them IC1 PCM3060PW

Commit message: Assign all footprints
Parts:
- removed C1, C3, C5: 10uF, symbol Device:CP1
- added C1, C3, C5: 10uF, Capacitor_SMD:C_0805_2012Metric, symbol Device:C
- C2, C4, C6: footprint (none) -> Capacitor_SMD:C_0805_2012Metric
Connections:
- net +3V3: now also C3.1
- net +5VA: now also C1.1
- net CODEC_VCOM: now also C5.1
- net GND: now also C1.2, C3.2, C5.2
Changed lines of the file:
@@
-	1    0    0    -1
-$EndComp
-$Comp
-L Device:CP1 C1
-U 1 1 6109A07D
-P 5000 1150
-F 0 "C1" H 4800 1200 50  0000 L CNN
-F 1 "10uF" H 4700 1100 50  0000 L CNN
-F 2 "" H 5000 1150 50  0001 C CNN
-F 3 "~" H 5000 1150 50  0001 C CNN
-	1    5000 1150
 	1    0    0    -1
 $EndComp
@@
 F 0 "C2" H 5365 1196 50  0000 L CNN
 F 1 "100nF" H 5365 1105 50  0000 L CNN
-F 2 "" H 5288 1000 50  0001 C CNN
+F 2 "Capacitor_SMD:C_0805_2012Metric" H 5288 1000 50  0001 C CNN
 F 3 "~" H 5250 1150 50  0001 C CNN
 	1    5250 1150
@@
 Wire Wire Line
 	5250 1300 5000 1300
-Connection ~ 5000 1300
 Text Label 1400 1550 2    50   ~ 0
 DGND
@@
 	1    0    0    -1
 $EndComp
-$Comp
-L Device:CP1 C3
-U 1 1 610DECD1
-P 6050 1150
-F 0 "C3" H 5850 1200 50  0000 L CNN
-F 1 "10uF" H 5750 1100 50  0000 L CNN
-F 2 "" H 6050 1150 50  0001 C CNN
-F 3 "~" H 6050 1150 50  0001 C CNN
-	1    6050 1150
-	1    0    0    -1
-$EndComp
 Wire Wire Line
 	6550 1000 6300 1000
@@
 	6300 1000 6050 1000
 Connection ~ 6300 1000
-Connection ~ 6050 1000
 $Comp
 L Device:C C4
@@
 F 0 "C4" H 6415 1196 50  0000 L CNN
 F 1 "100nF" H 6415 1105 50  0000 L CNN
-F 2 "" H 6338 1000 50  0001 C CNN
+F 2 "Capacitor_SMD:C_0805_2012Metric" H 6338 1000 50  0001 C CNN
 F 3 "~" H 6300 1150 50  0001 C CNN
 	1    6300 1150
@@
 Wire Wire Line
 	6300 1300 6050 1300
-Connection ~ 6050 1300
 $Comp
 L power:+5VA #PWR01
@@
 	1    0    0    -1
 $EndComp
-Connection ~ 5000 1000
 Text Label 3300 1550 0    50   ~ 0
 VCOM
 Text Label 7100 1000 2    50   ~ 0
 VCOM
-$Comp
-L Device:CP1 C5
-U 1 1 610E6A81
-P 7100 1150
-F 0 "C5" H 6900 1200 50  0000 L CNN
-F 1 "10uF" H 6800 1100 50  0000 L CNN
-F 2 "" H 7100 1150 50  0001 C CNN
-F 3 "~" H 7100 1150 50  0001 C CNN
-	1    7100 1150
-	1    0    0    -1
-$EndComp
 $Comp
 L Device:C C6
@@
 F 0 "C6" H 7465 1196 50  0000 L CNN
 F 1 "100nF" H 7465 1105 50  0000 L CNN
-F 2 "" H 7388 1000 50  0001 C CNN
+F 2 "Capacitor_SMD:C_0805_2012Metric" H 7388 1000 50  0001 C CNN
 F 3 "~" H 7350 1150 50  0001 C CNN
 	1    7350 1150
@@
 Wire Wire Line
 	7350 1300 7100 1300
-Connection ~ 7100 1300
 $Comp
 L power:GND #PWR05
@@
 Text Notes 6000 750  0    50   ~ 0
 12mA
+$Comp
+L Device:C C1
+U 1 1 611004AE
+P 5000 1150
+F 0 "C1" H 4800 1200 50  0000 L CNN
+F 1 "10uF" H 4700 1100 50  0000 L CNN
+F 2 "Capacitor_SMD:C_0805_2012Metric" H 5038 1000 50  0001 C CNN
+F 3 "~" H 5000 1150 50  0001 C CNN
+	1    5000 1150
+	1    0    0    -1
+$EndComp
+Connection ~ 5000 1000
+Connection ~ 5000 1300
+$Comp
+L Device:C C3
+U 1 1 61100675
+P 6050 1150
+F 0 "C3" H 5850 1200 50  0000 L CNN
+F 1 "10uF" H 5750 1100 50  0000 L CNN
+F 2 "Capacitor_SMD:C_0805_2012Metric" H 6088 1000 50  0001 C CNN
+F 3 "~" H 6050 1150 50  0001 C CNN
+	1    6050 1150
+	1    0    0    -1
+$EndComp
+Connection ~ 6050 1000
+Connection ~ 6050 1300
+$Comp
+L Device:C C5
+U 1 1 61100A3E
+P 7100 1150
+F 0 "C5" H 6900 1200 50  0000 L CNN
+F 1 "10uF" H 6800 1100 50  0000 L CNN
+F 2 "Capacitor_SMD:C_0805_2012Metric" H 7138 1000 50  0001 C CNN
+F 3 "~" H 7100 1150 50  0001 C CNN
+	1    7100 1150
+	1    0    0    -1
+$EndComp
+Connection ~ 7100 1300
 $EndSCHEMATC

Commit message: PCB layout work and related changes to the schematic
Parts:
- added TP1: PCM_CLK TP, TestPoint:TestPoint_Loop_D2.60mm_Drill1.6mm_Beaded, symbol Connector:TestPoint
- added TP2: PCM_FS TP, TestPoint:TestPoint_Loop_D2.60mm_Drill1.6mm_Beaded, symbol Connector:TestPoint
- added TP3: PCM_DIN TP, TestPoint:TestPoint_Loop_D2.60mm_Drill1.6mm_Beaded, symbol Connector:TestPoint
- added TP4: PCM_DOUT TP, TestPoint:TestPoint_Loop_D2.60mm_Drill1.6mm_Beaded, symbol Connector:TestPoint
- added TP5: CODEC_SDA TP, TestPoint:TestPoint_Loop_D2.60mm_Drill1.6mm_Beaded, symbol Connector:TestPoint
- added TP6: CODEC_SCL TP, TestPoint:TestPoint_Loop_D2.60mm_Drill1.6mm_Beaded, symbol Connector:TestPoint
Connections:
- net ADC_OUT renamed CM4_PCM_DIN
- net CM4_PCM_DIN: now also TP3.1
- net ADC_VIN_L renamed CODEC_VIN_L
- net ADC_VIN_R renamed CODEC_VIN_R
- net CODEC_BCK renamed CM4_PCM_CLK
- net CM4_PCM_CLK: now also TP1.1
- net CODEC_LRCK renamed CM4_PCM_FS
- net CM4_PCM_FS: now also TP2.1
- net CODEC_SCL renamed CM4_SCL0
- net CM4_SCL0: now also TP6.1
- net CODEC_SDA renamed CM4_SDA0
- net CM4_SDA0: now also TP5.1
- net DAC_IN renamed CM4_PCM_DOUT
- net CM4_PCM_DOUT: now also TP4.1
- net DAC_VOUT_L+ renamed CODEC_VOUT_L+
- net DAC_VOUT_L- renamed CODEC_VOUT_L-
- net DAC_VOUT_R+ renamed CODEC_VOUT_R+
- net DAC_VOUT_R- renamed CODEC_VOUT_R-
Other:
- note added: "CODEC interface"
- moved on the sheet: C1, C2, C3, C4, C5, C6, IC1
