File: Convolution Thing/Gates.sch (KiCad schematic (older format))
At the start: 17 parts

Commit message: Fix some issues, add component references
Parts:
- gave numbers to parts that had none: 17
Changed lines of the file:
@@
 $EndDescr
 $Comp
-L Device:Q_NPN_BEC Q?
+L Device:Q_NPN_BEC Q1
 U 1 1 610C1679
 P 1900 1700
-F 0 "Q?" H 2091 1746 50  0000 L CNN
+F 0 "Q1" H 2091 1746 50  0000 L CNN
 F 1 "NPN" H 2091 1655 50  0000 L CNN
 F 2 "" H 2100 1800 50  0001 C CNN
@@
 P 1100 1700
 AR Path="/61055545/610CBBF6" Ref="J?"  Part="1"
-AR Path="/610C04CE/610CBBF6" Ref="J?"  Part="1"
-F 0 "J?" H 921 1633 50  0000 R CNN
+AR Path="/610C04CE/610CBBF6" Ref="J18"  Part="1"
+F 0 "J18" H 921 1633 50  0000 R CNN
 F 1 "Gate In 1" H 1250 1400 50  0000 R CNN
 F 2 "" H 1100 1700 50  0001 C CNN
@@
 $EndComp
 $Comp
-L Device:R R?
+L Device:R R61
 U 1 1 610CCE9A
 P 1550 1700
-F 0 "R?" V 1450 1700 50  0000 C CNN
+F 0 "R61" V 1450 1700 50  0000 C CNN
 F 1 "100k" V 1550 1700 50  0000 C CNN
 F 2 "" V 1480 1700 50  0001 C CNN
@@
 	1400 1700 1300 1700
 $Comp
-L power:GND #PWR?
+L power:GND #PWR0130
 U 1 1 610CD1DC
 P 1300 1800
-F 0 "#PWR?" H 1300 1550 50  0001 C CNN
+F 0 "#PWR0130" H 1300 1550 50  0001 C CNN
 F 1 "GND" H 1305 1627 50  0000 C CNN
 F 2 "" H 1300 1800 50  0001 C CNN
@@
 $EndComp
 $Comp
-L power:GND #PWR?
+L power:GND #PWR0135
 U 1 1 610CE1C2
 P 2000 1900
-F 0 "#PWR?" H 2000 1650 50  0001 C CNN
+F 0 "#PWR0135" H 2000 1650 50  0001 C CNN
 F 1 "GND" H 2005 1727 50  0000 C CNN
 F 2 "" H 2000 1900 50  0001 C CNN
@@
 $EndComp
 $Comp
-L Device:R R?
+L Device:R R65
 U 1 1 610CF225
 P 2000 1150
-F 0 "R?" H 2070 1196 50  0000 L CNN
+F 0 "R65" H 2070 1196 50  0000 L CNN
 F 1 "10k" V 2000 1100 50  0000 L CNN
 F 2 "" V 1930 1150 50  0001 C CNN
@@
 $EndComp
 $Comp
-L power:+3.3V #PWR?
+L power:+3.3V #PWR0134
 U 1 1 610CF760
 P 2000 1000
-F 0 "#PWR?" H 2000 850 50  0001 C CNN
+F 0 "#PWR0134" H 2000 850 50  0001 C CNN
 F 1 "+3.3V" H 2015 1173 50  0000 C CNN
 F 2 "" H 2000 1000 50  0001 C CNN
@@
 Connection ~ 2000 1400
 $Comp
-L Device:Q_NPN_BEC Q?
+L Device:Q_NPN_BEC Q2
 U 1 1 610D3CCF
 P 1900 3300
-F 0 "Q?" H 2091 3346 50  0000 L CNN
+F 0 "Q2" H 2091 3346 50  0000 L CNN
 F 1 "NPN" H 2091 3255 50  0000 L CNN
 F 2 "" H 2100 3400 50  0001 C CNN
@@
 P 1100 3300
 AR Path="/61055545/610D3CD5" Ref="J?"  Part="1"
-AR Path="/610C04CE/610D3CD5" Ref="J?"  Part="1"
-F 0 "J?" H 921 3233 50  0000 R CNN
+AR Path="/610C04CE/610D3CD5" Ref="J19"  Part="1"
+F 0 "J19" H 921 3233 50  0000 R CNN
 F 1 "Gate In 2" H 1250 3000 50  0000 R CNN
 F 2 "" H 1100 3300 50  0001 C CNN
@@
 $EndComp
 $Comp
-L Device:R R?
+L Device:R R62
 U 1 1 610D3CDB
 P 1550 3300
-F 0 "R?" V 1450 3300 50  0000 C CNN
+F 0 "R62" V 1450 3300 50  0000 C CNN
 F 1 "100k" V 1550 3300 50  0000 C CNN
 F 2 "" V 1480 3300 50  0001 C CNN
@@
 	1400 3300 1300 3300
 $Comp
-L power:GND #PWR?
+L power:GND #PWR0131
 U 1 1 610D3CE2
 P 1300 3400
-F 0 "#PWR?" H 1300 3150 50  0001 C CNN
+F 0 "#PWR0131" H 1300 3150 50  0001 C CNN
 F 1 "GND" H 1305 3227 50  0000 C CNN
 F 2 "" H 1300 3400 50  0001 C CNN
@@
 $EndComp
 $Comp
-L power:GND #PWR?
+L power:GND #PWR0137
 U 1 1 610D3CE8
 P 2000 3500
-F 0 "#PWR?" H 2000 3250 50  0001 C CNN
+F 0 "#PWR0137" H 2000 3250 50  0001 C CNN
 F 1 "GND" H 2005 3327 50  0000 C CNN
 F 2 "" H 2000 3500 50  0001 C CNN
@@
 $EndComp
 $Comp
-L Device:R R?
+L Device:R R66
 U 1 1 610D3CEE
 P 2000 2750
-F 0 "R?" H 2070 2796 50  0000 L CNN
+F 0 "R66" H 2070 2796 50  0000 L CNN
 F 1 "10k" V 2000 2700 50  0000 L CNN
 F 2 "" V 1930 2750 50  0001 C CNN
@@
 $EndComp
 $Comp
-L power:+3.3V #PWR?
+L power:+3.3V #PWR0136
 U 1 1 610D3CF4
 P 2000 2600
-F 0 "#PWR?" H 2000 2450 50  0001 C CNN
+F 0 "#PWR0136" H 2000 2450 50  0001 C CNN
 F 1 "+3.3V" H 2015 2773 50  0000 C CNN
 F 2 "" H 2000 2600 50  0001 C CNN
@@
 Connection ~ 2000 3000
 $Comp
-L Device:Q_NPN_BEC Q?
+L Device:Q_NPN_BEC Q3
 U 1 1 610D42B8
 P 1900 4800
-F 0 "Q?" H 2091 4846 50  0000 L CNN
+F 0 "Q3" H 2091 4846 50  0000 L CNN
 F 1 "NPN" H 2091 4755 50  0000 L CNN
 F 2 "" H 2100 4900 50  0001 C CNN
@@
 P 1100 4800
 AR Path="/61055545/610D42BE" Ref="J?"  Part="1"
-AR Path="/610C04CE/610D42BE" Ref="J?"  Part="1"
-F 0 "J?" H 921 4733 50  0000 R CNN
+AR Path="/610C04CE/610D42BE" Ref="J20"  Part="1"
+F 0 "J20" H 921 4733 50  0000 R CNN
 F 1 "Gate In 3" H 1250 4500 50  0000 R CNN
 F 2 "" H 1100 4800 50  0001 C CNN
@@
 $EndComp
 $Comp
-L Device:R R?
+L Device:R R63
 U 1 1 610D42C4
 P 1550 4800
-F 0 "R?" V 1450 4800 50  0000 C CNN
+F 0 "R63" V 1450 4800 50  0000 C CNN
 F 1 "100k" V 1550 4800 50  0000 C CNN
 F 2 "" V 1480 4800 50  0001 C CNN
@@
 	1400 4800 1300 4800
 $Comp
-L power:GND #PWR?
+L power:GND #PWR0132
 U 1 1 610D42CB
 P 1300 4900
-F 0 "#PWR?" H 1300 4650 50  0001 C CNN
+F 0 "#PWR0132" H 1300 4650 50  0001 C CNN
 F 1 "GND" H 1305 4727 50  0000 C CNN
 F 2 "" H 1300 4900 50  0001 C CNN
@@
 $EndComp
 $Comp
-L power:GND #PWR?
+L power:GND #PWR0139
 U 1 1 610D42D1
 P 2000 5000
-F 0 "#PWR?" H 2000 4750 50  0001 C CNN
+F 0 "#PWR0139" H 2000 4750 50  0001 C CNN
 F 1 "GND" H 2005 4827 50  0000 C CNN
 F 2 "" H 2000 5000 50  0001 C CNN
@@
 $EndComp
 $Comp
-L Device:R R?
+L Device:R R67
 U 1 1 610D42D7
 P 2000 4250
-F 0 "R?" H 2070 4296 50  0000 L CNN
+F 0 "R67" H 2070 4296 50  0000 L CNN
 F 1 "10k" V 2000 4200 50  0000 L CNN
 F 2 "" V 1930 4250 50  0001 C CNN
@@
 $EndComp
 $Comp
-L power:+3.3V #PWR?
+L power:+3.3V #PWR0138
 U 1 1 610D42DD
 P 2000 4100
-F 0 "#PWR?" H 2000 3950 50  0001 C CNN
+F 0 "#PWR0138" H 2000 3950 50  0001 C CNN
 F 1 "+3.3V" H 2015 4273 50  0000 C CNN
 F 2 "" H 2000 4100 50  0001 C CNN
@@
 Connection ~ 2000 4500
 $Comp
-L Device:Q_NPN_BEC Q?
+L Device:Q_NPN_BEC Q4
 U 1 1 610D4866
 P 1900 6300
-F 0 "Q?" H 2091 6346 50  0000 L CNN
+F 0 "Q4" H 2091 6346 50  0000 L CNN
 F 1 "NPN" H 2091 6255 50  0000 L CNN
 F 2 "" H 2100 6400 50  0001 C CNN
@@
 P 1100 6300
 AR Path="/61055545/610D486C" Ref="J?"  Part="1"
-AR Path="/610C04CE/610D486C" Ref="J?"  Part="1"
-F 0 "J?" H 921 6233 50  0000 R CNN
+AR Path="/610C04CE/610D486C" Ref="J21"  Part="1"
+F 0 "J21" H 921 6233 50  0000 R CNN
 F 1 "Gate In 4" H 1250 6000 50  0000 R CNN
 F 2 "" H 1100 6300 50  0001 C CNN
@@
 $EndComp
 $Comp
-L Device:R R?
+L Device:R R64
 U 1 1 610D4872
 P 1550 6300
-F 0 "R?" V 1450 6300 50  0000 C CNN
+F 0 "R64" V 1450 6300 50  0000 C CNN
 F 1 "100k" V 1550 6300 50  0000 C CNN
 F 2 "" V 1480 6300 50  0001 C CNN
@@
 	1400 6300 1300 6300
 $Comp
-L power:GND #PWR?
+L power:GND #PWR0133
 U 1 1 610D4879
 P 1300 6400
-F 0 "#PWR?" H 1300 6150 50  0001 C CNN
+F 0 "#PWR0133" H 1300 6150 50  0001 C CNN
 F 1 "GND" H 1305 6227 50  0000 C CNN
 F 2 "" H 1300 6400 50  0001 C CNN
@@
 $EndComp
 $Comp
-L power:GND #PWR?
+L power:GND #PWR0141
 U 1 1 610D487F
 P 2000 6500
-F 0 "#PWR?" H 2000 6250 50  0001 C CNN
+F 0 "#PWR0141" H 2000 6250 50  0001 C CNN
 F 1 "GND" H 2005 6327 50  0000 C CNN
 F 2 "" H 2000 6500 50  0001 C CNN
@@
 $EndComp
 $Comp
-L Device:R R?
+L Device:R R68
 U 1 1 610D4885
 P 2000 5750
-F 0 "R?" H 2070 5796 50  0000 L CNN
+F 0 "R68" H 2070 5796 50  0000 L CNN
 F 1 "10k" V 2000 5700 50  0000 L CNN
 F 2 "" V 1930 5750 50  0001 C CNN
@@
 $EndComp
 $Comp
-L power:+3.3V #PWR?
+L power:+3.3V #PWR0140
 U 1 1 610D488B
 P 2000 5600
-F 0 "#PWR?" H 2000 5450 50  0001 C CNN
+F 0 "#PWR0140" H 2000 5450 50  0001 C CNN
 F 1 "+3.3V" H 2015 5773 50  0000 C CNN
 F 2 "" H 2000 5600 50  0001 C CNN
@@
 Connection ~ 2000 6000
 $Comp
-L Connector:TestPoint TP?
+L Connector:TestPoint TP20
 U 1 1 6117A11F
 P 2000 1400
-F 0 "TP?" V 2050 1650 50  0000 C CNN
+F 0 "TP20" V 2050 1650 50  0000 C CNN
 F 1 "Gate TP" V 1950 1750 50  0000 C CNN
 F 2 "" H 2200 1400 50  0001 C CNN

Commit message: Assign all footprints
Parts:
- J18, J19, J20, J21: footprint (none) -> SamacSys:ACJMNV352S
- Q1, Q2, Q3, Q4: footprint (none) -> Package_TO_SOT_SMD:SOT-23
- R57: renamed from R61; footprint (none) -> Resistor_SMD:R_0805_2012Metric
- R58: renamed from R62; footprint (none) -> Resistor_SMD:R_0805_2012Metric
- R59: renamed from R63; footprint (none) -> Resistor_SMD:R_0805_2012Metric
- R60: renamed from R64; footprint (none) -> Resistor_SMD:R_0805_2012Metric
- R61: renamed from R65; footprint (none) -> Resistor_SMD:R_0805_2012Metric
- R62: renamed from R66; footprint (none) -> Resistor_SMD:R_0805_2012Metric
- R63: renamed from R67; footprint (none) -> Resistor_SMD:R_0805_2012Metric
- R64: renamed from R68; footprint (none) -> Resistor_SMD:R_0805_2012Metric
- TP20: footprint (none) -> TestPoint:TestPoint_Loop_D2.60mm_Drill1.6mm_Beaded
Changed lines of the file:
@@
 F 0 "Q1" H 2091 1746 50  0000 L CNN
 F 1 "NPN" H 2091 1655 50  0000 L CNN
-F 2 "" H 2100 1800 50  0001 C CNN
+F 2 "Package_TO_SOT_SMD:SOT-23" H 2100 1800 50  0001 C CNN
 F 3 "~" H 1900 1700 50  0001 C CNN
 	1    1900 1700
@@
 F 0 "J18" H 921 1633 50  0000 R CNN
 F 1 "Gate In 1" H 1250 1400 50  0000 R CNN
-F 2 "" H 1100 1700 50  0001 C CNN
+F 2 "SamacSys:ACJMNV352S" H 1100 1700 50  0001 C CNN
 F 3 "~" H 1100 1700 50  0001 C CNN
 	1    1100 1700
@@
 $EndComp
 $Comp
-L Device:R R61
+L Device:R R57
 U 1 1 610CCE9A
 P 1550 1700
-F 0 "R61" V 1450 1700 50  0000 C CNN
+F 0 "R57" V 1450 1700 50  0000 C CNN
 F 1 "100k" V 1550 1700 50  0000 C CNN
-F 2 "" V 1480 1700 50  0001 C CNN
+F 2 "Resistor_SMD:R_0805_2012Metric" V 1480 1700 50  0001 C CNN
 F 3 "~" H 1550 1700 50  0001 C CNN
 	1    1550 1700
@@
 	1400 1700 1300 1700
 $Comp
-L power:GND #PWR0130
+L power:GND #PWR0123
 U 1 1 610CD1DC
 P 1300 1800
-F 0 "#PWR0130" H 1300 1550 50  0001 C CNN
+F 0 "#PWR0123" H 1300 1550 50  0001 C CNN
 F 1 "GND" H 1305 1627 50  0000 C CNN
 F 2 "" H 1300 1800 50  0001 C CNN
@@
 $EndComp
 $Comp
-L power:GND #PWR0135
+L power:GND #PWR0128
 U 1 1 610CE1C2
 P 2000 1900
-F 0 "#PWR0135" H 2000 1650 50  0001 C CNN
+F 0 "#PWR0128" H 2000 1650 50  0001 C CNN
 F 1 "GND" H 2005 1727 50  0000 C CNN
 F 2 "" H 2000 1900 50  0001 C CNN
@@
 $EndComp
 $Comp
-L Device:R R65
+L Device:R R61
 U 1 1 610CF225
 P 2000 1150
-F 0 "R65" H 2070 1196 50  0000 L CNN
+F 0 "R61" H 2070 1196 50  0000 L CNN
 F 1 "10k" V 2000 1100 50  0000 L CNN
-F 2 "" V 1930 1150 50  0001 C CNN
+F 2 "Resistor_SMD:R_0805_2012Metric" V 1930 1150 50  0001 C CNN
 F 3 "~" H 2000 1150 50  0001 C CNN
 	1    2000 1150
@@
 $EndComp
 $Comp
-L power:+3.3V #PWR0134
+L power:+3.3V #PWR0127
 U 1 1 610CF760
 P 2000 1000
-F 0 "#PWR0134" H 2000 850 50  0001 C CNN
+F 0 "#PWR0127" H 2000 850 50  0001 C CNN
 F 1 "+3.3V" H 2015 1173 50  0000 C CNN
 F 2 "" H 2000 1000 50  0001 C CNN
@@
 F 0 "Q2" H 2091 3346 50  0000 L CNN
 F 1 "NPN" H 2091 3255 50  0000 L CNN
-F 2 "" H 2100 3400 50  0001 C CNN
+F 2 "Package_TO_SOT_SMD:SOT-23" H 2100 3400 50  0001 C CNN
 F 3 "~" H 1900 3300 50  0001 C CNN
 	1    1900 3300
@@
 F 0 "J19" H 921 3233 50  0000 R CNN
 F 1 "Gate In 2" H 1250 3000 50  0000 R CNN
-F 2 "" H 1100 3300 50  0001 C CNN
+F 2 "SamacSys:ACJMNV352S" H 1100 3300 50  0001 C CNN
 F 3 "~" H 1100 3300 50  0001 C CNN
 	1    1100 3300
@@
 $EndComp
 $Comp
-L Device:R R62
+L Device:R R58
 U 1 1 610D3CDB
 P 1550 3300
-F 0 "R62" V 1450 3300 50  0000 C CNN
+F 0 "R58" V 1450 3300 50  0000 C CNN
 F 1 "100k" V 1550 3300 50  0000 C CNN
-F 2 "" V 1480 3300 50  0001 C CNN
+F 2 "Resistor_SMD:R_0805_2012Metric" V 1480 3300 50  0001 C CNN
 F 3 "~" H 1550 3300 50  0001 C CNN
 	1    1550 3300
@@
 	1400 3300 1300 3300
 $Comp
-L power:GND #PWR0131
+L power:GND #PWR0124
 U 1 1 610D3CE2
 P 1300 3400
-F 0 "#PWR0131" H 1300 3150 50  0001 C CNN
+F 0 "#PWR0124" H 1300 3150 50  0001 C CNN
 F 1 "GND" H 1305 3227 50  0000 C CNN
 F 2 "" H 1300 3400 50  0001 C CNN
@@
 $EndComp
 $Comp
-L power:GND #PWR0137
+L power:GND #PWR0130
 U 1 1 610D3CE8
 P 2000 3500
-F 0 "#PWR0137" H 2000 3250 50  0001 C CNN
+F 0 "#PWR0130" H 2000 3250 50  0001 C CNN
 F 1 "GND" H 2005 3327 50  0000 C CNN
 F 2 "" H 2000 3500 50  0001 C CNN
@@
 $EndComp
 $Comp
-L Device:R R66
+L Device:R R62
 U 1 1 610D3CEE
 P 2000 2750
-F 0 "R66" H 2070 2796 50  0000 L CNN
+F 0 "R62" H 2070 2796 50  0000 L CNN
 F 1 "10k" V 2000 2700 50  0000 L CNN
-F 2 "" V 1930 2750 50  0001 C CNN
+F 2 "Resistor_SMD:R_0805_2012Metric" V 1930 2750 50  0001 C CNN
 F 3 "~" H 2000 2750 50  0001 C CNN
 	1    2000 2750
@@
 $EndComp
 $Comp
-L power:+3.3V #PWR0136
+L power:+3.3V #PWR0129
 U 1 1 610D3CF4
 P 2000 2600
-F 0 "#PWR0136" H 2000 2450 50  0001 C CNN
+F 0 "#PWR0129" H 2000 2450 50  0001 C CNN
 F 1 "+3.3V" H 2015 2773 50  0000 C CNN
 F 2 "" H 2000 2600 50  0001 C CNN
@@
 F 0 "Q3" H 2091 4846 50  0000 L CNN
 F 1 "NPN" H 2091 4755 50  0000 L CNN
-F 2 "" H 2100 4900 50  0001 C CNN
+F 2 "Package_TO_SOT_SMD:SOT-23" H 2100 4900 50  0001 C CNN
 F 3 "~" H 1900 4800 50  0001 C CNN
 	1    1900 4800
@@
 F 0 "J20" H 921 4733 50  0000 R CNN
 F 1 "Gate In 3" H 1250 4500 50  0000 R CNN
-F 2 "" H 1100 4800 50  0001 C CNN
+F 2 "SamacSys:ACJMNV352S" H 1100 4800 50  0001 C CNN
 F 3 "~" H 1100 4800 50  0001 C CNN
 	1    1100 4800
@@
 $EndComp
 $Comp
-L Device:R R63
+L Device:R R59
 U 1 1 610D42C4
 P 1550 4800
-F 0 "R63" V 1450 4800 50  0000 C CNN
+F 0 "R59" V 1450 4800 50  0000 C CNN
 F 1 "100k" V 1550 4800 50  0000 C CNN
-F 2 "" V 1480 4800 50  0001 C CNN
+F 2 "Resistor_SMD:R_0805_2012Metric" V 1480 4800 50  0001 C CNN
 F 3 "~" H 1550 4800 50  0001 C CNN
 	1    1550 4800
@@
 	1400 4800 1300 4800
 $Comp
-L power:GND #PWR0132
+L power:GND #PWR0125
 U 1 1 610D42CB
 P 1300 4900
-F 0 "#PWR0132" H 1300 4650 50  0001 C CNN
+F 0 "#PWR0125" H 1300 4650 50  0001 C CNN
 F 1 "GND" H 1305 4727 50  0000 C CNN
 F 2 "" H 1300 4900 50  0001 C CNN
@@
 $EndComp
 $Comp
-L power:GND #PWR0139
+L power:GND #PWR0132
 U 1 1 610D42D1
 P 2000 5000
-F 0 "#PWR0139" H 2000 4750 50  0001 C CNN
+F 0 "#PWR0132" H 2000 4750 50  0001 C CNN
 F 1 "GND" H 2005 4827 50  0000 C CNN
 F 2 "" H 2000 5000 50  0001 C CNN
@@
 $EndComp
 $Comp
-L Device:R R67
+L Device:R R63
 U 1 1 610D42D7
 P 2000 4250
-F 0 "R67" H 2070 4296 50  0000 L CNN
+F 0 "R63" H 2070 4296 50  0000 L CNN
 F 1 "10k" V 2000 4200 50  0000 L CNN
-F 2 "" V 1930 4250 50  0001 C CNN
+F 2 "Resistor_SMD:R_0805_2012Metric" V 1930 4250 50  0001 C CNN
 F 3 "~" H 2000 4250 50  0001 C CNN
 	1    2000 4250
@@
 $EndComp
 $Comp
-L power:+3.3V #PWR0138
+L power:+3.3V #PWR0131
 U 1 1 610D42DD
 P 2000 4100
-F 0 "#PWR0138" H 2000 3950 50  0001 C CNN
+F 0 "#PWR0131" H 2000 3950 50  0001 C CNN
 F 1 "+3.3V" H 2015 4273 50  0000 C CNN
 F 2 "" H 2000 4100 50  0001 C CNN
@@
 F 0 "Q4" H 2091 6346 50  0000 L CNN
 F 1 "NPN" H 2091 6255 50  0000 L CNN
-F 2 "" H 2100 6400 50  0001 C CNN
+F 2 "Package_TO_SOT_SMD:SOT-23" H 2100 6400 50  0001 C CNN
 F 3 "~" H 1900 6300 50  0001 C CNN
 	1    1900 6300
@@
 F 0 "J21" H 921 6233 50  0000 R CNN
 F 1 "Gate In 4" H 1250 6000 50  0000 R CNN
-F 2 "" H 1100 6300 50  0001 C CNN
+F 2 "SamacSys:ACJMNV352S" H 1100 6300 50  0001 C CNN
 F 3 "~" H 1100 6300 50  0001 C CNN
 	1    1100 6300
@@
 $EndComp
 $Comp
-L Device:R R64
+L Device:R R60
 U 1 1 610D4872
 P 1550 6300
-F 0 "R64" V 1450 6300 50  0000 C CNN
+F 0 "R60" V 1450 6300 50  0000 C CNN
 F 1 "100k" V 1550 6300 50  0000 C CNN
-F 2 "" V 1480 6300 50  0001 C CNN
+F 2 "Resistor_SMD:R_0805_2012Metric" V 1480 6300 50  0001 C CNN
 F 3 "~" H 1550 6300 50  0001 C CNN
 	1    1550 6300
@@
 	1400 6300 1300 6300
 $Comp
-L power:GND #PWR0133
+L power:GND #PWR0126
 U 1 1 610D4879
 P 1300 6400
-F 0 "#PWR0133" H 1300 6150 50  0001 C CNN
+F 0 "#PWR0126" H 1300 6150 50  0001 C CNN
 F 1 "GND" H 1305 6227 50  0000 C CNN
 F 2 "" H 1300 6400 50  0001 C CNN
@@
 $EndComp
 $Comp
-L power:GND #PWR0141
+L power:GND #PWR0134
 U 1 1 610D487F
 P 2000 6500
-F 0 "#PWR0141" H 2000 6250 50  0001 C CNN
+F 0 "#PWR0134" H 2000 6250 50  0001 C CNN
 F 1 "GND" H 2005 6327 50  0000 C CNN
 F 2 "" H 2000 6500 50  0001 C CNN
@@
 $EndComp
 $Comp
-L Device:R R68
+L Device:R R64
 U 1 1 610D4885
 P 2000 5750
-F 0 "R68" H 2070 5796 50  0000 L CNN
+F 0 "R64" H 2070 5796 50  0000 L CNN
 F 1 "10k" V 2000 5700 50  0000 L CNN
-F 2 "" V 1930 5750 50  0001 C CNN
+F 2 "Resistor_SMD:R_0805_2012Metric" V 1930 5750 50  0001 C CNN
 F 3 "~" H 2000 5750 50  0001 C CNN
 	1    2000 5750
@@
 $EndComp
 $Comp
-L power:+3.3V #PWR0140
+L power:+3.3V #PWR0133
 U 1 1 610D488B
 P 2000 5600
-F 0 "#PWR0140" H 2000 5450 50  0001 C CNN
+F 0 "#PWR0133" H 2000 5450 50  0001 C CNN
 F 1 "+3.3V" H 2015 5773 50  0000 C CNN
 F 2 "" H 2000 5600 50  0001 C CNN
@@
 F 0 "TP20" V 2050 1650 50  0000 C CNN
 F 1 "Gate TP" V 1950 1750 50  0000 C CNN
-F 2 "" H 2200 1400 50  0001 C CNN
+F 2 "TestPoint:TestPoint_Loop_D2.60mm_Drill1.6mm_Beaded" H 2200 1400 50  0001 C CNN
 F 3 "~" H 2200 1400 50  0001 C CNN
 	1    2000 1400
