File: Convolution Thing/Gates.sch (KiCad schematic (older format))
At the start: 17 parts, among them J18 Gate In 1, J19 Gate In 2, J20 Gate In 3, J21 Gate In 4, Q1 NPN, Q2 NPN, Q3 NPN, Q4 NPN

Commit message: PCB layout work and related changes to the schematic
Parts:
- added TP28: Gate 2 TP, TestPoint:TestPoint_Loop_D2.60mm_Drill1.6mm_Beaded, symbol Connector:TestPoint
- added TP29: Gate 3 TP, TestPoint:TestPoint_Loop_D2.60mm_Drill1.6mm_Beaded, symbol Connector:TestPoint
- added TP30: Gate 4 TP, TestPoint:TestPoint_Loop_D2.60mm_Drill1.6mm_Beaded, symbol Connector:TestPoint
- J16: renamed from J18; footprint SamacSys:ACJMNV352S -> Connector_Audio:Jack_3.5mm_QingPu_WQP-PJ398SM_Vertical_CircularHoles
- J17: renamed from J19; footprint SamacSys:ACJMNV352S -> Connector_Audio:Jack_3.5mm_QingPu_WQP-PJ398SM_Vertical_CircularHoles
- J18: renamed from J20; footprint SamacSys:ACJMNV352S -> Connector_Audio:Jack_3.5mm_QingPu_WQP-PJ398SM_Vertical_CircularHoles
- J19: renamed from J21; footprint SamacSys:ACJMNV352S -> Connector_Audio:Jack_3.5mm_QingPu_WQP-PJ398SM_Vertical_CircularHoles
- TP27: renamed from TP20; value Gate TP -> Gate 1 TP
Connections:
- net GATE_IN_2: now also TP28.1
- net GATE_IN_3: now also TP29.1
- net GATE_IN_4: now also TP30.1
Changed lines of the file:
@@
 $Descr A4 11693 8268
 encoding utf-8
-Sheet 12 13
+Sheet 11 13
 Title ""
 Date ""
@@
 P 1100 1700
 AR Path="/61055545/610CBBF6" Ref="J?"  Part="1"
-AR Path="/610C04CE/610CBBF6" Ref="J18"  Part="1"
-F 0 "J18" H 921 1633 50  0000 R CNN
+AR Path="/610C04CE/610CBBF6" Ref="J16"  Part="1"
+F 0 "J16" H 921 1633 50  0000 R CNN
 F 1 "Gate In 1" H 1250 1400 50  0000 R CNN
-F 2 "SamacSys:ACJMNV352S" H 1100 1700 50  0001 C CNN
+F 2 "Connector_Audio:Jack_3.5mm_QingPu_WQP-PJ398SM_Vertical_CircularHoles" H 1100 1700 50  0001 C CNN
 F 3 "~" H 1100 1700 50  0001 C CNN
 	1    1100 1700
@@
 	1400 1700 1300 1700
 $Comp
-L power:GND #PWR0123
+L power:GND #PWR0113
 U 1 1 610CD1DC
 P 1300 1800
-F 0 "#PWR0123" H 1300 1550 50  0001 C CNN
+F 0 "#PWR0113" H 1300 1550 50  0001 C CNN
 F 1 "GND" H 1305 1627 50  0000 C CNN
 F 2 "" H 1300 1800 50  0001 C CNN
@@
 $EndComp
 $Comp
-L power:GND #PWR0128
+L power:GND #PWR0118
 U 1 1 610CE1C2
 P 2000 1900
-F 0 "#PWR0128" H 2000 1650 50  0001 C CNN
+F 0 "#PWR0118" H 2000 1650 50  0001 C CNN
 F 1 "GND" H 2005 1727 50  0000 C CNN
 F 2 "" H 2000 1900 50  0001 C CNN
@@
 $EndComp
 $Comp
-L power:+3.3V #PWR0127
+L power:+3.3V #PWR0117
 U 1 1 610CF760
 P 2000 1000
-F 0 "#PWR0127" H 2000 850 50  0001 C CNN
+F 0 "#PWR0117" H 2000 850 50  0001 C CNN
 F 1 "+3.3V" H 2015 1173 50  0000 C CNN
 F 2 "" H 2000 1000 50  0001 C CNN
@@
 	1    0    0    -1
 $EndComp
-Text GLabel 2100 1400 2    50   Output ~ 0
-GATE_IN_1
 Wire Wire Line
 	2100 1400 2000 1400
@@
 P 1100 3300
 AR Path="/61055545/610D3CD5" Ref="J?"  Part="1"
-AR Path="/610C04CE/610D3CD5" Ref="J19"  Part="1"
-F 0 "J19" H 921 3233 50  0000 R CNN
+AR Path="/610C04CE/610D3CD5" Ref="J17"  Part="1"
+F 0 "J17" H 921 3233 50  0000 R CNN
 F 1 "Gate In 2" H 1250 3000 50  0000 R CNN
-F 2 "SamacSys:ACJMNV352S" H 1100 3300 50  0001 C CNN
+F 2 "Connector_Audio:Jack_3.5mm_QingPu_WQP-PJ398SM_Vertical_CircularHoles" H 1100 3300 50  0001 C CNN
 F 3 "~" H 1100 3300 50  0001 C CNN
 	1    1100 3300
@@
 	1400 3300 1300 3300
 $Comp
-L power:GND #PWR0124
+L power:GND #PWR0114
 U 1 1 610D3CE2
 P 1300 3400
-F 0 "#PWR0124" H 1300 3150 50  0001 C CNN
+F 0 "#PWR0114" H 1300 3150 50  0001 C CNN
 F 1 "GND" H 1305 3227 50  0000 C CNN
 F 2 "" H 1300 3400 50  0001 C CNN
@@
 $EndComp
 $Comp
-L power:GND #PWR0130
+L power:GND #PWR0120
 U 1 1 610D3CE8
 P 2000 3500
-F 0 "#PWR0130" H 2000 3250 50  0001 C CNN
+F 0 "#PWR0120" H 2000 3250 50  0001 C CNN
 F 1 "GND" H 2005 3327 50  0000 C CNN
 F 2 "" H 2000 3500 50  0001 C CNN
@@
 $EndComp
 $Comp
-L power:+3.3V #PWR0129
+L power:+3.3V #PWR0119
 U 1 1 610D3CF4
 P 2000 2600
-F 0 "#PWR0129" H 2000 2450 50  0001 C CNN
+F 0 "#PWR0119" H 2000 2450 50  0001 C CNN
 F 1 "+3.3V" H 2015 2773 50  0000 C CNN
 F 2 "" H 2000 2600 50  0001 C CNN
@@
 	1    0    0    -1
 $EndComp
-Text GLabel 2100 3000 2    50   Output ~ 0
-GATE_IN_2
 Wire Wire Line
 	2100 3000 2000 3000
@@
 P 1100 4800
 AR Path="/61055545/610D42BE" Ref="J?"  Part="1"
-AR Path="/610C04CE/610D42BE" Ref="J20"  Part="1"
-F 0 "J20" H 921 4733 50  0000 R CNN
+AR Path="/610C04CE/610D42BE" Ref="J18"  Part="1"
+F 0 "J18" H 921 4733 50  0000 R CNN
 F 1 "Gate In 3" H 1250 4500 50  0000 R CNN
-F 2 "SamacSys:ACJMNV352S" H 1100 4800 50  0001 C CNN
+F 2 "Connector_Audio:Jack_3.5mm_QingPu_WQP-PJ398SM_Vertical_CircularHoles" H 1100 4800 50  0001 C CNN
 F 3 "~" H 1100 4800 50  0001 C CNN
 	1    1100 4800
@@
 	1400 4800 1300 4800
 $Comp
-L power:GND #PWR0125
+L power:GND #PWR0115
 U 1 1 610D42CB
 P 1300 4900
-F 0 "#PWR0125" H 1300 4650 50  0001 C CNN
+F 0 "#PWR0115" H 1300 4650 50  0001 C CNN
 F 1 "GND" H 1305 4727 50  0000 C CNN
 F 2 "" H 1300 4900 50  0001 C CNN
@@
 $EndComp
 $Comp
-L power:GND #PWR0132
+L power:GND #PWR0122
 U 1 1 610D42D1
 P 2000 5000
-F 0 "#PWR0132" H 2000 4750 50  0001 C CNN
+F 0 "#PWR0122" H 2000 4750 50  0001 C CNN
 F 1 "GND" H 2005 4827 50  0000 C CNN
 F 2 "" H 2000 5000 50  0001 C CNN
@@
 $EndComp
 $Comp
-L power:+3.3V #PWR0131
+L power:+3.3V #PWR0121
 U 1 1 610D42DD
 P 2000 4100
-F 0 "#PWR0131" H 2000 3950 50  0001 C CNN
+F 0 "#PWR0121" H 2000 3950 50  0001 C CNN
 F 1 "+3.3V" H 2015 4273 50  0000 C CNN
 F 2 "" H 2000 4100 50  0001 C CNN
@@
 	1    0    0    -1
 $EndComp
-Text GLabel 2100 4500 2    50   Output ~ 0
-GATE_IN_3
 Wire Wire Line
 	2100 4500 2000 4500
@@
 P 1100 6300
 AR Path="/61055545/610D486C" Ref="J?"  Part="1"
-AR Path="/610C04CE/610D486C" Ref="J21"  Part="1"
-F 0 "J21" H 921 6233 50  0000 R CNN
+AR Path="/610C04CE/610D486C" Ref="J19"  Part="1"
+F 0 "J19" H 921 6233 50  0000 R CNN
 F 1 "Gate In 4" H 1250 6000 50  0000 R CNN
-F 2 "SamacSys:ACJMNV352S" H 1100 6300 50  0001 C CNN
+F 2 "Connector_Audio:Jack_3.5mm_QingPu_WQP-PJ398SM_Vertical_CircularHoles" H 1100 6300 50  0001 C CNN
 F 3 "~" H 1100 6300 50  0001 C CNN
 	1    1100 6300
@@
 	1400 6300 1300 6300
 $Comp
-L power:GND #PWR0126
+L power:GND #PWR0116
 U 1 1 610D4879
 P 1300 6400
-F 0 "#PWR0126" H 1300 6150 50  0001 C CNN
+F 0 "#PWR0116" H 1300 6150 50  0001 C CNN
 F 1 "GND" H 1305 6227 50  0000 C CNN
 F 2 "" H 1300 6400 50  0001 C CNN
@@
 $EndComp
 $Comp
-L power:GND #PWR0134
+L power:GND #PWR0124
 U 1 1 610D487F
 P 2000 6500
-F 0 "#PWR0134" H 2000 6250 50  0001 C CNN
+F 0 "#PWR0124" H 2000 6250 50  0001 C CNN
 F 1 "GND" H 2005 6327 50  0000 C CNN
 F 2 "" H 2000 6500 50  0001 C CNN
@@
 $EndComp
 $Comp
-L power:+3.3V #PWR0133
+L power:+3.3V #PWR0123
 U 1 1 610D488B
 P 2000 5600
-F 0 "#PWR0133" H 2000 5450 50  0001 C CNN
+F 0 "#PWR0123" H 2000 5450 50  0001 C CNN
 F 1 "+3.3V" H 2015 5773 50  0000 C CNN
 F 2 "" H 2000 5600 50  0001 C CNN
@@
 	1    0    0    -1
 $EndComp
-Text GLabel 2100 6000 2    50   Output ~ 0
-GATE_IN_4
 Wire Wire Line
 	2100 6000 2000 6000
@@
 Connection ~ 2000 6000
 $Comp
-L Connector:TestPoint TP20
+L Connector:TestPoint TP27
 U 1 1 6117A11F
 P 2000 1400
-F 0 "TP20" V 2050 1650 50  0000 C CNN
-F 1 "Gate TP" V 1950 1750 50  0000 C CNN
+F 0 "TP27" V 2050 1650 50  0000 C CNN
+F 1 "Gate 1 TP" V 1950 1750 50  0000 C CNN
 F 2 "TestPoint:TestPoint_Loop_D2.60mm_Drill1.6mm_Beaded" H 2200 1400 50  0001 C CNN
 F 3 "~" H 2200 1400 50  0001 C CNN
@@
 NoConn ~ 1300 4700
 NoConn ~ 1300 6200
+$Comp
+L Connector:TestPoint TP28
+U 1 1 6115FAEE
+P 2000 3000
+F 0 "TP28" V 2050 3250 50  0000 C CNN
+F 1 "Gate 2 TP" V 1950 3350 50  0000 C CNN
+F 2 "TestPoint:TestPoint_Loop_D2.60mm_Drill1.6mm_Beaded" H 2200 3000 50  0001 C CNN
+F 3 "~" H 2200 3000 50  0001 C CNN
+	1    2000 3000
+	0    -1   -1   0
+$EndComp
+$Comp
+L Connector:TestPoint TP29
+U 1 1 61160006
+P 2000 4500
+F 0 "TP29" V 2050 4750 50  0000 C CNN
+F 1 "Gate 3 TP" V 1950 4850 50  0000 C CNN
+F 2 "TestPoint:TestPoint_Loop_D2.60mm_Drill1.6mm_Beaded" H 2200 4500 50  0001 C CNN
+F 3 "~" H 2200 4500 50  0001 C CNN
+	1    2000 4500
+	0    -1   -1   0
+$EndComp
+$Comp
+L Connector:TestPoint TP30
+U 1 1 611600DB
+P 2000 6000
+F 0 "TP30" V 2050 6250 50  0000 C CNN
+F 1 "Gate 4 TP" V 1950 6350 50  0000 C CNN
+F 2 "TestPoint:TestPoint_Loop_D2.60mm_Drill1.6mm_Beaded" H 2200 6000 50  0001 C CNN
+F 3 "~" H 2200 6000 50  0001 C CNN
+	1    2000 6000
+	0    -1   -1   0
+$EndComp
+Text GLabel 2100 6000 2    50   Output ~ 0
+GATE_IN_4
+Text GLabel 2100 4500 2    50   Output ~ 0
+GATE_IN_3
+Text GLabel 2100 3000 2    50   Output ~ 0
+GATE_IN_2
+Text GLabel 2100 1400 2    50   Output ~ 0
+GATE_IN_1
 $EndSCHEMATC
