File: Convolution Thing/LEDs.sch (KiCad schematic (older format))
At the start: 7 parts, among them IC3 LP55231, J16 LED Header

Commit message: PCB layout work and related changes to the schematic
Parts:
- removed J16: LED Header, Connector_PinHeader_2.54mm:PinHeader_1x09_P2.54mm_Vertical, symbol Connector:Conn_01x09_Female
- added C63: 100nF, Capacitor_SMD:C_0805_2012Metric, symbol Device:C
- added D10: LED 7, LED_SMD:LED_0805_2012Metric, symbol Device:LED
- added D11: LED 8, LED_SMD:LED_0805_2012Metric, symbol Device:LED
- added D12: LED 9, LED_SMD:LED_0805_2012Metric, symbol Device:LED
- added D13: Activity LED, LED_SMD:LED_0805_2012Metric, symbol Device:LED
- added D14: Power LED, LED_SMD:LED_0805_2012Metric, symbol Device:LED
- added D4: LED 1, LED_SMD:LED_0805_2012Metric, symbol Device:LED
- added D5: LED 2, LED_SMD:LED_0805_2012Metric, symbol Device:LED
- added D6: LED 3, LED_SMD:LED_0805_2012Metric, symbol Device:LED
- added D7: LED 4, LED_SMD:LED_0805_2012Metric, symbol Device:LED
- added D8: LED 5, LED_SMD:LED_0805_2012Metric, symbol Device:LED
- added D9: LED 6, LED_SMD:LED_0805_2012Metric, symbol Device:LED
- added IC3: SN74LVC1G07DCK3, SamacSys:SOT65P210X110-5N, symbol SamacSys:SN74LVC1G07DCK3
- added R55, R56: 100, Resistor_SMD:R_0805_2012Metric, symbol Device:R
- added TP25: LED_SCL TP, TestPoint:TestPoint_Loop_D2.60mm_Drill1.6mm_Beaded, symbol Connector:TestPoint
- added TP26: LED_SDA TP, TestPoint:TestPoint_Loop_D2.60mm_Drill1.6mm_Beaded, symbol Connector:TestPoint
- renumbered C62 to C58, C63 to C59, C64 to C60, C65 to C61, C66 to C62, IC3 to IC2
Connections:
- net D1: now also D4.2 (A)
- net D2: now also D5.2 (A)
- net D3: now also D6.2 (A)
- net D4: now also D7.2 (A)
- net D5: now also D8.2 (A)
- net D6: now also D9.2 (A)
- net D7: now also D10.2 (A)
- net D8: now also D11.2 (A)
- net D9: now also D12.2 (A)
- net GND: now also C63.2, D10.1 (K), D11.1 (K), D12.1 (K), D4.1 (K), D5.1 (K), D6.1 (K), D7.1 (K), D8.1 (K), D9.1 (K), IC3.3 (GND)
- net LED_SCL renamed CM4_SCL4
- net CM4_SCL4: now also TP25.1
- net LED_SDA renamed CM4_SDA4
- net CM4_SDA4: now also TP26.1
- new net: D13.1 (K), R55.1
- new net: IC3.4 (Y), R56.2
- new net: D14.1 (K), R56.1
- new net +3V3: C63.1, D13.2 (A), D14.2 (A), IC3.5 (VCC)
- new net CM4_LED_ACTIVITY: R55.2
- new net CM4_LED_POWER: IC3.2 (A)
