File: Convolution Thing/PSU.sch (KiCad schematic (older format))
At the start: 21 parts, among them J1 Eurorack power, J2 Power Header, U1 Compute_Module_4_Functional, U2 TLV1117-50, U3 ADP2303ARDZ-5.0

Commit message: Started footprint assignment
Parts:
- U1: value Compute_Module_4_Functional -> Compute Module 4; footprint (none) -> CM4:Raspberry-Pi-4-Compute-Module
Changed lines of the file:
@@
 P 950 2700
 F 0 "U1" H 1800 2997 60  0000 C CNN
-F 1 "Compute_Module_4_Functional" H 1800 2891 60  0000 C CNN
-F 2 "" H 1150 2750 60  0001 L CNN
+F 1 "Compute Module 4" H 1800 2891 60  0000 C CNN
+F 2 "CM4:Raspberry-Pi-4-Compute-Module" H 1150 2750 60  0001 L CNN
 F 3 "" H 1150 2550 60  0001 L CNN
 	1    950  2700

Commit message: Assign all footprints
Parts:
- removed C13: 100uf, symbol Device:CP1
- removed C14: 10uF, symbol Device:CP1
- removed C8: 10uf, symbol Device:CP1
- added C13: 100uF, Capacitor_SMD:C_1210_3225Metric, symbol Device:C
- added C14, C8: 10uF, Capacitor_SMD:C_0805_2012Metric, symbol Device:C
- added C16: 47uF, Capacitor_SMD:C_0805_2012Metric, symbol Device:C
- C10, C11, C12, C15, C7, C9: footprint (none) -> Capacitor_SMD:C_0805_2012Metric
- D1, D2, D3: footprint (none) -> Diode_SMD:D_SOD-123
- J1: footprint (none) -> Connector_PinHeader_2.54mm:PinHeader_2x10_P2.54mm_Vertical_SMD
- J2: footprint (none) -> Connector_PinSocket_2.54mm:PinSocket_1x04_P2.54mm_Vertical
- L1: value 10uH -> 4.7uH; footprint (none) -> Inductor_SMD:L_Vishay_IHLP-2020
- R1: footprint (none) -> Resistor_SMD:R_0805_2012Metric
- TP1, TP2: footprint (none) -> TestPoint:TestPoint_Loop_D2.60mm_Drill1.6mm_Beaded
- U2: footprint (none) -> Package_TO_SOT_SMD:SOT-223
Connections:
- net +12V: now also C8.1
- net +3V3: now also C14.1
- net +5V: now also C16.1
- net +5VA: now also C13.1
- net GND: now also C13.2, C14.2, C16.2, C8.2
Other:
- moved on the sheet: TP2
Changed lines of the file:
@@
 F 0 "J1" H 1200 1250 50  0000 C CNN
 F 1 "Eurorack power" H 1200 1850 50  0000 C CNN
-F 2 "" H 1150 1550 50  0001 C CNN
+F 2 "Connector_PinHeader_2.54mm:PinHeader_2x10_P2.54mm_Vertical_SMD" H 1150 1550 50  0001 C CNN
 F 3 "~" H 1150 1550 50  0001 C CNN
 	1    1150 1550
@@
 F 0 "D1" H 1700 933 50  0000 C CNN
 F 1 "Schottky" H 1700 1024 50  0000 C CNN
-F 2 "" H 1700 1150 50  0001 C CNN
+F 2 "Diode_SMD:D_SOD-123" H 1700 1150 50  0001 C CNN
 F 3 "~" H 1700 1150 50  0001 C CNN
 	1    1700 1150
@@
 F 0 "D2" H 1700 1750 50  0000 C CNN
 F 1 "Schottky" H 1700 1850 50  0000 C CNN
-F 2 "" H 1700 1950 50  0001 C CNN
+F 2 "Diode_SMD:D_SOD-123" H 1700 1950 50  0001 C CNN
 F 3 "~" H 1700 1950 50  0001 C CNN
 	1    1700 1950
@@
 NoConn ~ 2650 3000
 NoConn ~ 2650 3100
-$Comp
-L Device:CP1 C14
-U 1 1 61086D1E
-P 3000 2950
-F 0 "C14" H 2800 2900 50  0000 L CNN
-F 1 "10uF" H 3115 2905 50  0000 L CNN
-F 2 "" H 3000 2950 50  0001 C CNN
-F 3 "~" H 3000 2950 50  0001 C CNN
-	1    3000 2950
-	1    0    0    -1
-$EndComp
-Connection ~ 3000 2800
 Wire Wire Line
 	1950 1950 2400 1950
@@
 F 0 "C11" H 2065 1396 50  0000 L CNN
 F 1 "22uF" H 2065 1305 50  0000 L CNN
-F 2 "" H 1950 1350 50  0001 C CNN
+F 2 "Capacitor_SMD:C_0805_2012Metric" H 1950 1350 50  0001 C CNN
 F 3 "~" H 1950 1350 50  0001 C CNN
 	1    1950 1350
@@
 F 0 "C12" H 2065 1796 50  0000 L CNN
 F 1 "22uF" H 2065 1705 50  0000 L CNN
-F 2 "" H 1950 1750 50  0001 C CNN
+F 2 "Capacitor_SMD:C_0805_2012Metric" H 1950 1750 50  0001 C CNN
 F 3 "~" H 1950 1750 50  0001 C CNN
 	1    1950 1750
@@
 F 0 "TP1" V 2950 4300 50  0000 L CNN
 F 1 "+5VA TP" V 2850 4400 50  0000 L CNN
-F 2 "" H 3050 4200 50  0001 C CNN
+F 2 "TestPoint:TestPoint_Loop_D2.60mm_Drill1.6mm_Beaded" H 3050 4200 50  0001 C CNN
 F 3 "~" H 3050 4200 50  0001 C CNN
 	1    2850 4200
 	0    1    1    0
 $EndComp
-Connection ~ 2500 4200
 $Comp
 L power:GND #PWR022
@@
 	1    0    0    -1
 $EndComp
-Wire Wire Line
-	2250 4200 2500 4200
-Wire Wire Line
-	2850 4200 2500 4200
 $Comp
 L power:GND #PWR014
@@
 	1    0    0    -1
 $EndComp
-Wire Wire Line
-	950  4200 1100 4200
-$Comp
-L Device:CP1 C8
-U 1 1 610C12F0
-P 1100 4350
-F 0 "C8" H 850 4400 50  0000 L CNN
-F 1 "10uf" H 800 4300 50  0000 L CNN
-F 2 "" H 1100 4350 50  0001 C CNN
-F 3 "~" H 1100 4350 50  0001 C CNN
-	1    1100 4350
-	1    0    0    -1
-$EndComp
-Connection ~ 1100 4200
-$Comp
-L Device:CP1 C13
-U 1 1 610C12F8
-P 2500 4350
-F 0 "C13" H 2650 4400 50  0000 L CNN
-F 1 "100uf" H 2650 4300 50  0000 L CNN
-F 2 "" H 2500 4350 50  0001 C CNN
-F 3 "~" H 2500 4350 50  0001 C CNN
-	1    2500 4350
-	1    0    0    -1
-$EndComp
 $Comp
 L Regulator_Linear:TLV1117-50 U2
@@
 F 0 "U2" H 1950 4442 50  0000 C CNN
 F 1 "TLV1117-50" H 1950 4351 50  0000 C CNN
-F 2 "" H 1950 4200 50  0001 C CNN
+F 2 "Package_TO_SOT_SMD:SOT-223" H 1950 4200 50  0001 C CNN
 F 3 "http://www.ti.com/lit/ds/symlink/tlv1117.pdf" H 1950 4200 50  0001 C CNN
 	1    1950 4200
@@
 F 0 "J2" H 4228 1226 50  0000 L CNN
 F 1 "Power Header" H 4228 1135 50  0000 L CNN
-F 2 "" H 4200 1250 50  0001 C CNN
+F 2 "Connector_PinSocket_2.54mm:PinSocket_1x04_P2.54mm_Vertical" H 4200 1250 50  0001 C CNN
 F 3 "~" H 4200 1250 50  0001 C CNN
 	1    4200 1250
@@
 $EndComp
 $Comp
-L power:+12V #PWR029
+L power:+12V #PWR028
 U 1 1 6110F9DD
 P 3800 1250
-F 0 "#PWR029" H 3800 1100 50  0001 C CNN
+F 0 "#PWR028" H 3800 1100 50  0001 C CNN
 F 1 "+12V" H 3815 1423 50  0000 C CNN
 F 2 "" H 3800 1250 50  0001 C CNN
@@
 F 0 "C7" H 800 3050 50  0000 L CNN
 F 1 "100nF" H 500 3050 50  0000 L CNN
-F 2 "" H 788 2800 50  0001 C CNN
+F 2 "Capacitor_SMD:C_0805_2012Metric" H 788 2800 50  0001 C CNN
 F 3 "~" H 750 2950 50  0001 C CNN
 	1    750  2950
@@
 F 0 "R1" H 1700 5750 50  0000 L CNN
 F 1 "100k" V 1600 5700 50  0000 L CNN
-F 2 "" V 1530 5800 50  0001 C CNN
+F 2 "Resistor_SMD:R_0805_2012Metric" V 1530 5800 50  0001 C CNN
 F 3 "~" H 1600 5800 50  0001 C CNN
 	1    1600 5800
@@
 F 0 "C15" V 2748 5600 50  0000 C CNN
 F 1 "100nF" V 2839 5600 50  0000 C CNN
-F 2 "" H 3038 5450 50  0001 C CNN
+F 2 "Capacitor_SMD:C_0805_2012Metric" H 3038 5450 50  0001 C CNN
 F 3 "~" H 3000 5600 50  0001 C CNN
 	1    3000 5600
@@
 F 0 "C9" H 1050 5850 50  0000 L CNN
 F 1 "100nF" H 950 5750 50  0000 L CNN
-F 2 "" H 1338 5650 50  0001 C CNN
+F 2 "Capacitor_SMD:C_0805_2012Metric" H 1338 5650 50  0001 C CNN
 F 3 "~" H 1300 5800 50  0001 C CNN
 	1    1300 5800
@@
 	2850 6000 2850 5800
 $Comp
-L power:+5V #PWR028
+L power:+5V #PWR032
 U 1 1 6128BF09
-P 3750 5600
-F 0 "#PWR028" H 3750 5450 50  0001 C CNN
-F 1 "+5V" H 3765 5773 50  0000 C CNN
-F 2 "" H 3750 5600 50  0001 C CNN
-F 3 "" H 3750 5600 50  0001 C CNN
-	1    3750 5600
-	1    0    0    -1
-$EndComp
-Text Notes 3700 5350 0    50   ~ 0
+P 4100 5600
+F 0 "#PWR032" H 4100 5450 50  0001 C CNN
+F 1 "+5V" H 4115 5773 50  0000 C CNN
+F 2 "" H 4100 5600 50  0001 C CNN
+F 3 "" H 4100 5600 50  0001 C CNN
+	1    4100 5600
+	1    0    0    -1
+$EndComp
+Text Notes 4050 5350 0    50   ~ 0
 3A
 $Comp
@@
 P 3450 5800
 F 0 "L1" H 3450 6015 50  0000 C CNN
-F 1 "10uH" H 3450 5924 50  0000 C CNN
-F 2 "" H 3450 5800 50  0001 C CNN
+F 1 "4.7uH" H 3450 5924 50  0000 C CNN
+F 2 "Inductor_SMD:L_Vishay_IHLP-2020" H 3450 5800 50  0001 C CNN
 F 3 "~" H 3450 5800 50  0001 C CNN
 	1    3450 5800
@@
 F 0 "D3" V 3104 6030 50  0000 L CNN
 F 1 "Catch Diode" V 3195 6030 50  0000 L CNN
-F 2 "" H 3150 5950 50  0001 C CNN
+F 2 "Diode_SMD:D_SOD-123" H 3150 5950 50  0001 C CNN
 F 3 "~" H 3150 5950 50  0001 C CNN
 	1    3150 5950
@@
 $EndComp
 Wire Wire Line
-	3750 5800 3700 5800
-Wire Wire Line
 	3150 5800 3200 5800
 Text Notes 700  2400 0    50   ~ 0
@@
 L Connector:TestPoint TP2
 U 1 1 612A8F5A
-P 3750 5800
-F 0 "TP2" V 3850 5900 50  0000 L CNN
-F 1 "+5V TP" V 3750 6000 50  0000 L CNN
-F 2 "" H 3950 5800 50  0001 C CNN
-F 3 "~" H 3950 5800 50  0001 C CNN
-	1    3750 5800
+P 4100 5800
+F 0 "TP2" V 4200 5900 50  0000 L CNN
+F 1 "+5V TP" V 4100 6000 50  0000 L CNN
+F 2 "TestPoint:TestPoint_Loop_D2.60mm_Drill1.6mm_Beaded" H 4300 5800 50  0001 C CNN
+F 3 "~" H 4300 5800 50  0001 C CNN
+	1    4100 5800
 	0    1    1    0
 $EndComp
-Connection ~ 3750 5800
-Wire Wire Line
-	3750 5600 3750 5800
+Wire Wire Line
+	4100 5600 4100 5800
 $Comp
 L Device:C C10
@@
 F 0 "C10" H 1465 4396 50  0000 L CNN
 F 1 "100nF" H 1450 4300 50  0000 L CNN
-F 2 "" H 1388 4200 50  0001 C CNN
+F 2 "Capacitor_SMD:C_0805_2012Metric" H 1388 4200 50  0001 C CNN
 F 3 "~" H 1350 4350 50  0001 C CNN
 	1    1350 4350
 	1    0    0    -1
 $EndComp
-Wire Wire Line
-	1100 4200 1350 4200
 Connection ~ 1350 4200
 $Comp
@@
 L power:PWR_FLAG #FLG04
 U 1 1 610F6B04
-P 3800 5600
-F 0 "#FLG04" H 3800 5675 50  0001 C CNN
-F 1 "PWR_FLAG" V 3800 5728 50  0000 L CNN
-F 2 "" H 3800 5600 50  0001 C CNN
-F 3 "~" H 3800 5600 50  0001 C CNN
-	1    3800 5600
+P 4150 5600
+F 0 "#FLG04" H 4150 5675 50  0001 C CNN
+F 1 "PWR_FLAG" V 4150 5728 50  0000 L CNN
+F 2 "" H 4150 5600 50  0001 C CNN
+F 3 "~" H 4150 5600 50  0001 C CNN
+	1    4150 5600
 	0    1    1    0
 $EndComp
 Wire Wire Line
-	3800 5600 3750 5600
-Connection ~ 3750 5600
+	4150 5600 4100 5600
+Connection ~ 4100 5600
+$Comp
+L Device:C C14
+U 1 1 611039B9
+P 3000 2950
+F 0 "C14" H 3115 2996 50  0000 L CNN
+F 1 "10uF" H 3115 2905 50  0000 L CNN
+F 2 "Capacitor_SMD:C_0805_2012Metric" H 3038 2800 50  0001 C CNN
+F 3 "~" H 3000 2950 50  0001 C CNN
+	1    3000 2950
+	1    0    0    -1
+$EndComp
+Connection ~ 3000 2800
+Wire Wire Line
+	950  4200 1100 4200
+$Comp
+L Device:C C8
+U 1 1 61104ABC
+P 1100 4350
+F 0 "C8" H 900 4400 50  0000 L CNN
+F 1 "10uF" H 800 4300 50  0000 L CNN
+F 2 "Capacitor_SMD:C_0805_2012Metric" H 1138 4200 50  0001 C CNN
+F 3 "~" H 1100 4350 50  0001 C CNN
+	1    1100 4350
+	1    0    0    -1
+$EndComp
+Connection ~ 1100 4200
+Wire Wire Line
+	1100 4200 1350 4200
+Wire Wire Line
+	2250 4200 2500 4200
+$Comp
+L Device:C C13
+U 1 1 61106112
+P 2500 4350
+F 0 "C13" H 2300 4300 50  0000 L CNN
+F 1 "100uF" H 2600 4300 50  0000 L CNN
+F 2 "Capacitor_SMD:C_1210_3225Metric" H 2538 4200 50  0001 C CNN
+F 3 "~" H 2500 4350 50  0001 C CNN
+	1    2500 4350
+	1    0    0    -1
+$EndComp
+Connection ~ 2500 4200
+Wire Wire Line
+	2500 4200 2850 4200
+$Comp
+L Device:C C16
+U 1 1 6117EAE1
+P 3900 5950
+F 0 "C16" H 4015 5996 50  0000 L CNN
+F 1 "47uF" H 4015 5905 50  0000 L CNN
+F 2 "Capacitor_SMD:C_0805_2012Metric" H 3938 5800 50  0001 C CNN
+F 3 "~" H 3900 5950 50  0001 C CNN
+	1    3900 5950
+	1    0    0    -1
+$EndComp
+Wire Wire Line
+	3900 5800 3700 5800
+Wire Wire Line
+	4100 5800 3900 5800
+Connection ~ 4100 5800
+Connection ~ 3900 5800
+$Comp
+L power:GND #PWR029
+U 1 1 61183F70
+P 3900 6100
+F 0 "#PWR029" H 3900 5850 50  0001 C CNN
+F 1 "GND" H 3905 5927 50  0000 C CNN
+F 2 "" H 3900 6100 50  0001 C CNN
+F 3 "" H 3900 6100 50  0001 C CNN
+	1    3900 6100
+	1    0    0    -1
+$EndComp
 $EndSCHEMATC

Commit message: PCB layout work and related changes to the schematic
Parts:
- removed C14: 10uF, Capacitor_SMD:C_0805_2012Metric, symbol Device:C
- removed C7: 100nF, Capacitor_SMD:C_0805_2012Metric, symbol Device:C
- removed U1: Compute Module 4, CM4:Raspberry-Pi-4-Compute-Module, symbol CM4:Compute_Module_4_Functional
- J1: footprint Connector_PinHeader_2.54mm:PinHeader_2x10_P2.54mm_Vertical_SMD -> Connector_PinHeader_2.54mm:PinHeader_2x05_P2.54mm_Vertical_SMD
- renumbered C11 to C10, C12 to C11, C13 to C12, C15 to C13, C16 to C14, C8 to C7, C9 to C8, C10 to C9, TP1 to TP7, TP2 to TP8, U2 to U1, U3 to U2
Connections:
- net +12V: now also J2.3 (Pin_3); no longer J2.2 (Pin_2)
- net +3V3: now also J2.4 (Pin_4); no longer J2.1 (Pin_1)
- net -12V: now also J2.2 (Pin_2); no longer J2.3 (Pin_3)
- net GND: now also J2.1 (Pin_1); no longer J2.4 (Pin_4)
- no-connect marks 2 -> 0
Other:
- note removed: "1.4A"
- note removed: "600mA"
- moved on the sheet: C12, C13, C14, C7, C8, C9, D3, L1, R1, TP7, TP8, U1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
